File: Habitat_V5/Habitat_V5.kicad_pcb (KiCad board)
At the start: 2 copper layers, 123 parts, among them J1 Conn_01x03_Socket, J2 Conn_01x03_Socket, J3 Conn_01x12, J4 Conn_01x03_Socket, J5 Conn_01x04_Socket, K1 Relay_SPDT, Q1 PMOS, Q2 2N7002K, Q3 40N02, U1 XL1509-5V, U11 ADS1115IDGS, U2 AP2112K-3.3, U3 PC817, U6 ESP32-WROOM-32

Commit message: Current update
Parts:
- removed C21: 100uF, Capacitor_SMD:C_Elec_6.3x7.7
- removed J1: Conn_01x03_Socket, Connector_JST:JST_NV_B03P-NV_1x03_P5.00mm_Vertical
- added D19: BAT54S, Package_TO_SOT_SMD:SOT-23, F.Cu at (140.0, 88.5)
- added D20: BAT54S, Package_TO_SOT_SMD:SOT-23, F.Cu at (140.1, 82.1)
- added H1: MountingHole, MountingHole:MountingHole_3.2mm_M3, F.Cu at (72.0, 47.0)
- added H2: MountingHole, MountingHole:MountingHole_3.2mm_M3, F.Cu at (67.8, 170.0)
- added H3: MountingHole, MountingHole:MountingHole_3.2mm_M3, F.Cu at (153.0, 170.0)
- added H4: MountingHole, MountingHole:MountingHole_3.2mm_M3, F.Cu at (153.0, 47.0)
- added R29: 10k, Resistor_SMD:R_0805_2012Metric, F.Cu at (83.4, 86.8)
- added R30: 10k, Resistor_SMD:R_0805_2012Metric, F.Cu at (83.4, 102.0)
- added R31: 10k, Resistor_SMD:R_0805_2012Metric, F.Cu at (83.6, 117.2)
- added R32: 10k, Resistor_SMD:R_0805_2012Metric, F.Cu at (83.6, 132.6)
- added R33: 10k, Resistor_SMD:R_0805_2012Metric, F.Cu at (83.4, 147.8)
- added R34: 10k, Resistor_SMD:R_0805_2012Metric, F.Cu at (83.6, 163.0)
- added RTC1: Conn_01x04_Socket, Library:RTC, F.Cu at (113.0, 97.2)
- added Relay1: Conn_01x03_Socket, TerminalBlock_Phoenix:TerminalBlock_Phoenix_MKDS-1,5-3_1x03_P5.00mm_Horizontal, F.Cu at (135.2, 166.2)
- CD6: value 100n -> 10u
- CD7: value 10u -> 100n
- D16: value 1N4148W -> BAT54S; footprint Diode_SMD:D_SOD-123 -> Package_TO_SOT_SMD:SOT-23
- D18: value BAT54S -> 1N4148W; footprint Package_TO_SOT_SMD:SOT-23 -> Diode_SMD:D_SOD-123
- J2, J4, PWM1: footprint TerminalBlock:TerminalBlock_Xinya_XY308-2.54-3P_1x03_P2.54mm_Horizontal -> TerminalBlock_Phoenix:TerminalBlock_Phoenix_MKDS-1,5-3_1x03_P5.00mm_Horizontal
- J5: value Conn_01x04_Socket -> Conn_01x03_Socket; footprint TerminalBlock_Phoenix:TerminalBlock_Phoenix_MKDS-3-5-5.08_1x05_P5.08mm_Horizontal -> TerminalBlock_Phoenix:TerminalBlock_Phoenix_MKDS-1,5-3_1x03_P5.00mm_Horizontal
- JP1: value SolderJumper_2_Open -> SolderJumper_3_Open; footprint Jumper:SolderJumper-2_P1.3mm_Open_RoundedPad1.0x1.5mm -> Jumper:SolderJumper-3_P2.0mm_Open_TrianglePad1.0x1.5mm
- JP2: value SolderJumper_3_Open -> SolderJumper_2_Open; footprint Jumper:SolderJumper-3_P2.0mm_Open_TrianglePad1.0x1.5mm -> Jumper:SolderJumper-2_P1.3mm_Open_RoundedPad1.0x1.5mm
- R26: value 8.2k -> 10k
- moved D15 142.9 mm to (71.6, 159.2), turned to -90 degrees
- moved C23 141.3 mm to (77.3, 155.1), turned to -90 degrees
- moved D13 139.8 mm to (71.6, 144.0), turned to -90 degrees
- moved C22 136.8 mm to (92.7, 156.6)
- moved D12 134.9 mm to (71.7, 128.8), turned to -90 degrees
- moved D2 133.3 mm to (63.5, 56.9), turned to 90 degrees
- moved D10 130.7 mm to (71.8, 113.4), turned to -90 degrees
- moved C24 130.4 mm to (84.7, 155.1), turned to -90 degrees
- moved D14 129.0 mm to (95.4, 164.2), turned to 90 degrees
- moved D3 128.9 mm to (65.8, 66.3), turned to -90 degrees
- moved CD3 128.0 mm to (83.3, 54.4)
- moved D9 127.5 mm to (71.7, 98.4), turned to -90 degrees
- moved D16 127.3 mm to (98.0, 88.3), turned to -90 degrees
- moved U10 125.7 mm to (77.7, 162.6), turned to -90 degrees
- moved D8 124.9 mm to (71.7, 83.0), turned to -90 degrees
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Connections:
- C1 pad 1: +5V -> +5V_H
- CD3 pad 1: +5V -> +5V_H
- D1 pad 1: +5V -> +5V_H
- D16 pad 1: +5V -> GND
- D16 pad 2: Net-(D16-A) -> +3.3V
- D17 pad 3: Net-(D17-COM) -> Rlevel
- D18 pad 1: GND -> +5V
- D18 pad 2: +3.3V -> Net-(D18-A)
- D4 pad 2: Vin -> VCC
- D5 pad 1: Vin -> VCC
- J5 pad 3: GPIO32 -> GND
- JP1 pad 1: Net-(JP1-A) -> +3.3V
- JP1 pad 2: V3 -> Net-(J5-Pin_1)
- JP2 pad 1: +3.3V -> Net-(JP2-A)
- JP2 pad 2: Net-(J5-Pin_1) -> V3
- K1 pad A1: Vin -> Net-(D5-A)
- K1 pad A2: Net-(D5-A) -> VCC
- R23 pad 1: Net-(D17-COM) -> Net-(D16-COM)
- R25 pad 2: Net-(D17-COM) -> Net-(D16-COM)
- R26 pad 1: Net-(D17-COM) -> GND
- R26 pad 2: GND -> Net-(D16-COM)
- R27 pad 2: Net-(JP1-A) -> Net-(JP2-A)
- SERIAL1 pad 1: Net-(D16-A) -> Net-(D18-A)
- SHT40 pad 2: SDA -> GND
- SHT40 pad 4: GND -> SDA
Routing:
- net VCC: track 0.00 -> 216.6 mm
- net +3.3V: track 0.00 -> 122.8 mm, vias 0 -> 2
- net EN_CH6: track 0.00 -> 89.2 mm, vias 0 -> 2
- net EN_CH5: track 0.00 -> 81.7 mm, vias 0 -> 2
- net EN_CH4: track 0.00 -> 71.0 mm, vias 0 -> 2
- net EN_CH7: track 0.00 -> 58.9 mm
- net EN_CH3: track 0.00 -> 52.6 mm, vias 0 -> 2
- net +5V_H: track 0.00 -> 49.7 mm, vias 0 -> 6
- net EN_CH2: track 0.00 -> 44.0 mm, vias 0 -> 2
- net Net-(U6-EN): track 0.00 -> 29.1 mm, vias 0 -> 2
- net PCH3: track 0.00 -> 27.5 mm
- net PCH2: track 0.00 -> 27.5 mm
- net PCH6: track 0.00 -> 27.5 mm
- net PCH5: track 0.00 -> 27.5 mm
- net PCH4: track 0.00 -> 27.5 mm
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- added copper zone on B.Cu, net GND
- added copper zone on F.Cu, net GND
Other:
- board outline added: 104.6 x 131 mm
- board text added: "0~3V3"
- board text added: "30~300R"
- board text added: "3V3 1W GND"
- board text added: "I2C 3V3"
- board text added: "I2C 5V"
- board text added: "Level + -"
- board text added: "Level2 + -"
- board text added: "NO C NC"
- board text added: "V3 + -"
- board text added: "VCC PWM GND"

Commit message: Updated PCB and Schematic
Parts:
- removed C27: 100n, Capacitor_SMD:C_0805_2012Metric
- removed the D14 at (95.4, 164.2)
- removed the D17 at (140.1, 94.9)
- removed the J5 at (148.8, 130.8)
- removed JP2: SolderJumper_2_Open, Jumper:SolderJumper-2_P1.3mm_Open_RoundedPad1.0x1.5mm
- removed the R19 at (106.4, 148.5)
- removed the R22 at (140.0, 97.7)
- removed the R27 at (136.7, 85.3)
- added D16: SS14, Diode_SMD:D_SMA, F.Cu at (92.0, 158.8)
- added D18: BAT54S, Package_TO_SOT_SMD:SOT-23, F.Cu at (134.9, 89.6)
- added J1: Conn_01x04_Socket, Connector_Phoenix_MSTB:PhoenixContact_MSTBA_2,5_4-G-5,08_1x04_P5.08mm_Horizontal, F.Cu at (60.8, 83.2)
- added J4: Conn_01x04_Socket, Connector_Phoenix_MSTB:PhoenixContact_MSTBA_2,5_4-G-5,08_1x04_P5.08mm_Horizontal, F.Cu at (60.8, 143.8)
- added Opto1: Conn_01x02_Pin, Connector_Phoenix_MSTB:PhoenixContact_MSTBA_2,5_2-G-5,08_1x02_P5.08mm_Horizontal, F.Cu at (144.4, 130.2)
- added Q10: 2N7002K, Package_TO_SOT_SMD:SOT-23, F.Cu at (119.1, 86.9)
- added Q11: 2N7002K, Package_TO_SOT_SMD:SOT-23, F.Cu at (123.1, 86.9)
- added Q12: 2N7002K, Package_TO_SOT_SMD:SOT-23, F.Cu at (102.4, 82.7)
- added Q13: 2N7002K, Package_TO_SOT_SMD:SOT-23, F.Cu at (106.2, 82.7)
- added Q14: 2N7002K, Package_TO_SOT_SMD:SOT-23, F.Cu at (110.1, 82.7)
- added Q15: 2N7002K, Package_TO_SOT_SMD:SOT-23, F.Cu at (114.2, 82.5)
- added Q16: 2N7002K, Package_TO_SOT_SMD:SOT-23, F.Cu at (118.2, 82.5)
- added Q17: 2N7002K, Package_TO_SOT_SMD:SOT-23, F.Cu at (122.2, 82.5)
- added Q4: 2N7002K, Package_TO_SOT_SMD:SOT-23, F.Cu at (108.0, 146.9)
- added Q5: 2N7002K, Package_TO_SOT_SMD:SOT-23, F.Cu at (104.2, 148.7)
- added Q6: 2N7002K, Package_TO_SOT_SMD:SOT-23, F.Cu at (103.3, 86.9)
- added Q7: 2N7002K, Package_TO_SOT_SMD:SOT-23, F.Cu at (107.2, 86.9)
- added Q8: 2N7002K, Package_TO_SOT_SMD:SOT-23, F.Cu at (111.1, 86.9)
- added Q9: 2N7002K, Package_TO_SOT_SMD:SOT-23, F.Cu at (115.1, 86.9)
- added R20: 10k, Resistor_SMD:R_0805_2012Metric, F.Cu at (111.5, 147.8)
- added R23: 2k2, Resistor_SMD:R_0805_2012Metric, F.Cu at (100.2, 148.7)
- added R25: 100k, Resistor_SMD:R_0805_2012Metric, F.Cu at (109.1, 149.8)
- added R26: 10k, Resistor_SMD:R_0805_2012Metric, F.Cu at (108.0, 143.8)
- added R29: 330, Resistor_SMD:R_0805_2012Metric, F.Cu at (134.9, 113.6)
- added R30: 10k, Resistor_SMD:R_0805_2012Metric, F.Cu at (103.2, 90.8)
- added R31: 10k, Resistor_SMD:R_0805_2012Metric, F.Cu at (107.2, 90.7)
- added R32: 10k, Resistor_SMD:R_0805_2012Metric, F.Cu at (111.0, 90.7)
- added R33: 10k, Resistor_SMD:R_0805_2012Metric, F.Cu at (115.0, 90.7)
- added R34: 10k, Resistor_SMD:R_0805_2012Metric, F.Cu at (119.0, 90.7)
- added R35: 10k, Resistor_SMD:R_0805_2012Metric, F.Cu at (123.0, 90.7)
- added R36: 10k, Resistor_SMD:R_0805_2012Metric, F.Cu at (126.9, 86.0)
- added R37: 10k, Resistor_SMD:R_0805_2012Metric, F.Cu at (102.4, 79.6)
- added R38: 10k, Resistor_SMD:R_0805_2012Metric, F.Cu at (106.3, 79.6)
- added R39: 10k, Resistor_SMD:R_0805_2012Metric, F.Cu at (110.1, 79.6)
- added R40: 10k, Resistor_SMD:R_0805_2012Metric, F.Cu at (114.2, 79.6)
- added R41: 10k, Resistor_SMD:R_0805_2012Metric, F.Cu at (118.2, 79.6)
- added R42: 10k, Resistor_SMD:R_0805_2012Metric, F.Cu at (122.2, 79.6)
- J2, Relay1: footprint TerminalBlock_Phoenix:TerminalBlock_Phoenix_MKDS-1,5-3_1x03_P5.00mm_Horizontal -> Connector_Phoenix_MSTB:PhoenixContact_MSTBA_2,5_3-G-5,08_1x03_P5.08mm_Horizontal
- J3: value Conn_01x12 -> Conn_01x04_Socket; footprint Connector_Phoenix_GMSTB:PhoenixContact_GMSTBVA_2,5_12-G-7,62_1x12_P7.62mm_Vertical -> Connector_Phoenix_MSTB:PhoenixContact_MSTBA_2,5_4-G-5,08_1x04_P5.08mm_Horizontal
- J5: renamed from J4; footprint TerminalBlock_Phoenix:TerminalBlock_Phoenix_MKDS-1,5-3_1x03_P5.00mm_Horizontal -> Connector_Phoenix_MSTB:PhoenixContact_MSTBA_2,5_3-G-5,08_1x03_P5.08mm_Horizontal
- JP1: value SolderJumper_3_Open -> SolderJumper_2_Open; footprint Jumper:SolderJumper-3_P2.0mm_Open_TrianglePad1.0x1.5mm -> Jumper:SolderJumper-2_P1.3mm_Open_RoundedPad1.0x1.5mm
- PWM1: value Conn_01x03_Socket -> Conn_01x02_Pin; footprint TerminalBlock_Phoenix:TerminalBlock_Phoenix_MKDS-1,5-3_1x03_P5.00mm_Horizontal -> Connector_Phoenix_MSTB:PhoenixContact_MSTBA_2,5_2-G-5,08_1x02_P5.08mm_Horizontal
- R24: value 330 -> 2k2
- R28: value 2k2 -> 330
- S1: renamed from B1; footprint Connector_Molex:Molex_KK-254_AE-6410-02A_1x02_P2.54mm_Vertical -> Connector_Phoenix_MSTB:PhoenixContact_MSTBA_2,5_2-G-5,08_1x02_P5.08mm_Horizontal
- S2: renamed from B2; footprint Connector_Molex:Molex_KK-254_AE-6410-02A_1x02_P2.54mm_Vertical -> Connector_Phoenix_MSTB:PhoenixContact_MSTBA_2,5_2-G-5,08_1x02_P5.08mm_Horizontal
- TH1: renamed from B3; footprint Connector_Molex:Molex_KK-254_AE-6410-02A_1x02_P2.54mm_Vertical -> Connector_Phoenix_MSTB:PhoenixContact_MSTBA_2,5_2-G-5,08_1x02_P5.08mm_Horizontal
- U6: value ESP32-WROOM-32 -> ESP32-S3-WROOM-1; footprint RF_Module:ESP32-WROOM-32 -> RF_Module:ESP32-S3-WROOM-1
- VDC1: footprint Connector_Phoenix_GMSTB:PhoenixContact_GMSTBVA_2,5_2-G-7,62_1x02_P7.62mm_Vertical -> Connector_Phoenix_MSTB:PhoenixContact_MSTBA_2,5_2-G-5,08_1x02_P5.08mm_Horizontal
- moved CD4 80.6 mm to (117.2, 142.1), turned to -90 degrees
- moved OLED1 78.5 mm to (115.4, 136.1)
- moved JP1 38.4 mm to (135.2, 92.8), turned to 0 degrees
- moved J3 35.9 mm to (60.8, 113.8)
- moved D19 28.5 mm to (134.9, 116.6)
- moved C26 28.5 mm to (99.8, 91.4), turned to 0 degrees
- moved S1 22.3 mm to (144.4, 116.8)
- moved D20 21.5 mm to (134.9, 103.0)
- moved C7 16.3 mm to (108.0, 74.1), turned to -90 degrees
- moved S2 15.3 mm to (144.4, 103.2)
- moved R24 11.0 mm to (131.7, 92.8), turned to 0 degrees
- moved R28 9.67 mm to (134.9, 100.0)
- moved CD6 9.00 mm to (137.8, 82.1), turned to 90 degrees
- moved D2 8.97 mm to (71.0, 52.0), turned to 180 degrees
- moved TH1 8.83 mm to (144.4, 89.8)
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- renumbered C18 to C19, C19 to C20, C20 to C21, C25 to C22, C22 to C23, C23 to C24, C24 to C25, CD7 to CD6, CD6 to CD7, D15 to D14, D18 to D15, D16 to D17, R16 to R15, R15 to R16, R21 to R19, R23 to R21, R25 to R22, R26 to R27, R9 to R7, R7 to R8, R8 to R9, SHT40 to SHT1
Connections:
- net /3V3MCU renamed 3V3MCU
- net Net-(U6-EN) renamed EN
- C8 pad 1: Net-(U6-IO0) -> PROG
- D19 pad 3: V2 -> V1
- D20 pad 3: V3 -> V2
- J3 pad 1: PCH1 -> PCH3
- J3 pad 2: NCH1 -> NCH3
- J3 pad 3: PCH2 -> PCH4
- J3 pad 4: NCH2 -> NCH4
- JP1 pad 1: +3.3V -> Net-(JP1-A)
- JP1 pad 2: Net-(J5-Pin_1) -> V3
- OLED2 pad 2: GPIO32 -> GPIO11
- OLED2 pad 3: GPIO33 -> GPIO10
- PROG1 pad 2: Net-(U6-IO0) -> PROG
- R13 pad 1: +3.3V -> PROG
- R13 pad 2: Net-(U6-IO0) -> +3.3V
- R24 pad 1: Rlevel -> +3.3V
- R24 pad 2: V1 -> Net-(JP1-A)
- R5 pad 2: GPIO33 -> GPIO10
- R6 pad 2: GPIO32 -> GPIO11
- S1 pad 1: Rlevel -> V1
- U6 pad 10: EN_CH7 -> unconnected-(U6-IO17-Pad10)
- U6 pad 11: Relay -> unconnected-(U6-IO18-Pad11)
- U6 pad 12: Opto -> GPIO10
- U6 pad 14: Neopixel -> unconnected-(U6-USB_D+-Pad14)
- U6 pad 15: GND -> unconnected-(U6-IO3-Pad15)
- U6 pad 16: EN_CH1 -> unconnected-(U6-IO46-Pad16)
- U6 pad 17: unconnected-(U6-SHD/SD2-Pad17) -> GPIO11
- U6 pad 18: unconnected-(U6-SWP/SD3-Pad18) -> SCL
- U6 pad 19: unconnected-(U6-SCS/CMD-Pad19) -> SDA
- U6 pad 20: unconnected-(U6-SCK/CLK-Pad20) -> Opto
- U6 pad 21: unconnected-(U6-SDO/SD0-Pad21) -> 1Wire
- U6 pad 22: unconnected-(U6-SDI/SD1-Pad22) -> CH7
- U6 pad 23: unconnected-(U6-IO15-Pad23) -> Relay
- U6 pad 25: Net-(U6-IO0) -> unconnected-(U6-IO48-Pad25)
- U6 pad 26: 1Wire -> unconnected-(U6-IO45-Pad26)
- U6 pad 27: EN_CH2 -> PROG
- U6 pad 28: EN_CH3 -> unconnected-(U6-IO35-Pad28)
- U6 pad 30: EN_CH4 -> unconnected-(U6-IO37-Pad30)
- U6 pad 31: EN_CH5 -> EN_MASTER
- U6 pad 33: SDA -> unconnected-(U6-IO40-Pad33)
- U6 pad 34: RX0 -> unconnected-(U6-IO41-Pad34)
- U6 pad 35: TX0 -> unconnected-(U6-IO42-Pad35)
- U6 pad 36: SCL -> RX0
- U6 pad 37: EN_CH6 -> TX0
- U6 pad 38: GND -> unconnected-(U6-IO2-Pad38)
- U6 pad 39: GND -> unconnected-(U6-IO1-Pad39)
- U6 pad 4: A0 -> CH1
- U6 pad 5: unconnected-(U6-SENSOR_VN-Pad5) -> CH2
- U6 pad 6: unconnected-(U6-IO34-Pad6) -> CH3
- U6 pad 7: unconnected-(U6-IO35-Pad7) -> CH4
- U6 pad 8: GPIO32 -> CH5
- U6 pad 9: GPIO33 -> CH6
- VDC1 pad 1: Vin -> GND
- VDC1 pad 2: GND -> Vin
Routing:
- net +3.3V: track 122.8 -> 402.4 mm, vias 2 -> 11
- net EN_MASTER: track 0.00 -> 119.1 mm, vias 0 -> 9
- net 1Wire: track 0.00 -> 111.0 mm, vias 0 -> 1
- net +5V: track 12.1 -> 118.1 mm, vias 0 -> 2
- net Relay: track 0.00 -> 102.0 mm, vias 0 -> 2
- net CH7: track 0.00 -> 101.0 mm, vias 0 -> 2
- net VCC: track 216.6 -> 289.4 mm
- net SDA: track 18.5 -> 77.9 mm, vias 0 -> 3
- net EN_CH7: track 58.9 -> 0.00 mm
- net SCL: track 23.3 -> 79.9 mm, vias 2 -> 3
- net V1: track 0.00 -> 44.1 mm
- net V0: track 0.00 -> 43.1 mm
- net CH6: track 0.00 -> 38.4 mm
- net CH5: track 0.00 -> 37.1 mm
- net CH4: track 0.00 -> 34.5 mm
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Other:
- board size 104.6 x 131 mm -> 100.6 x 131 mm
- board text added: "+Level1-"
- board text added: "+Level2-"
- board text added: "+V3-"
- board text added: "3V3"
- board text added: "VCC PWM"
- board text removed: "0~3V3"
- board text removed: "30~300R"
- board text removed: "Level + -"
- board text removed: "Level2 + -"
- board text removed: "V3 + -"
- board text removed: "VCC PWM GND"

Commit message: Validation pre fab
Pls check
Parts:
- removed the R20 at (101.1, 151.8)
- removed the R29 at (83.4, 86.8)
- removed the R30 at (83.4, 102.0)
- removed the R31 at (83.6, 117.2)
- removed the R32 at (83.6, 132.6)
- removed the R33 at (83.4, 147.8)
- removed the R34 at (83.6, 163.0)
- R17: value 0R22 -> 0R25
- moved R1 10.6 mm to (64.7, 61.6), turned to 180 degrees
- moved D2 9.72 mm to (69.5, 61.6)
- moved R15 5.90 mm to (86.9, 71.1)
- moved H1 5.00 mm to (67.0, 47.0)
- moved C22 4.53 mm to (119.5, 156.4), turned to 180 degrees
- moved C26 4.29 mm to (96.6, 94.2), turned to -90 degrees
- moved R7 2.83 mm to (149.1, 137.4), turned to 180 degrees
- moved D11 1.85 mm to (82.2, 72.0), turned to 0 degrees
- moved R27 1.83 mm to (93.9, 93.5), turned to 0 degrees
- moved Q1 1.54 mm to (67.7, 56.6), turned to 180 degrees
- moved VDC1 1.46 mm to (60.6, 51.5)
- moved R10 1.02 mm to (147.3, 139.8)
- moved Q2 1.00 mm to (147.2, 143.1)
- moved H2 0.80 mm to (67.0, 170.0)
- moved J5 0.24 mm to (111.7, 165.6)
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Connections:
- J5 pad 1: +3.3V -> GND
- J5 pad 3: GND -> +3.3V
- U6 pad 15: unconnected-(U6-IO3-Pad15) -> Neopixel
Routing:
- net +3.3V: track 402.4 -> 318.0 mm, vias 11 -> 7
- net Opto: track 7.64 -> 69.8 mm, vias 0 -> 2
- net GND: track 0.03 -> 42.2 mm, vias 18 -> 272
- net SCL: track 79.9 -> 117.7 mm, vias 3 -> 4
- net SDA: track 77.9 -> 115.1 mm, vias 3 -> 4
- net Neopixel: track 17.9 -> 46.8 mm, vias 0 -> 2
- net +5V: track 118.1 -> 145.0 mm, vias 2 -> 4
- net VCC: track 289.4 -> 276.6 mm
- net NCH2: track 24.4 -> 36.2 mm, vias 0 -> 1
- net NCH4: track 24.4 -> 35.3 mm, vias 0 -> 1
- net NCH6: track 25.0 -> 35.4 mm, vias 0 -> 1
- net EN_CH3: track 56.4 -> 47.3 mm
- net NCH3: track 20.9 -> 28.8 mm, vias 0 -> 1
- net 1Wire: track 111.0 -> 118.2 mm, vias 1 -> 2
- net NCH1: track 20.8 -> 27.9 mm, vias 0 -> 1
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Other:
- board text added: "GND 1W 3V3"
- board text removed: "3V3 1W GND"

Commit message: Review for production
Parts:
- R18: value 0R22 -> 0R25
- renumbered VDC2 to VDC1, VDC1 to VDC2
Connections:
- net GPIO10 renamed GPIO8
- net GPIO11 renamed GPIO9
- U6 pad 10: unconnected-(U6-IO17-Pad10) -> Neopixel
- U6 pad 15: Neopixel -> unconnected-(U6-IO3-Pad15)
Routing:
- net Neopixel: track 46.8 -> 43.3 mm

Commit message: Files for production
Parts:
- added CD8: 10u, Capacitor_SMD:C_0805_2012Metric, F.Cu at (140.2, 78.8)
- added JP2: SolderJumper_2_Open, Jumper:SolderJumper-2_P1.3mm_Open_RoundedPad1.0x1.5mm, F.Cu at (140.6, 91.0)
- added R25: 10k, Resistor_SMD:R_0805_2012Metric, F.Cu at (140.6, 87.3)
- added R27: 10k, Resistor_SMD:R_0805_2012Metric, F.Cu at (138.2, 85.4)
- Opto1: value Conn_01x02_Pin -> Conn_01x03_Pin; footprint Connector_Phoenix_MSTB:PhoenixContact_MSTBA_2,5_2-G-5,08_1x02_P5.08mm_Horizontal -> Connector_Phoenix_MSTB:PhoenixContact_MSTBA_2,5_3-G-5,08_1x03_P5.08mm_Horizontal
- moved SERIAL1 5.01 mm to (143.2, 57.2), turned to 90 degrees
- moved R21 4.05 mm to (134.9, 90.3), turned to 180 degrees
- moved CD6 3.28 mm to (137.8, 78.8)
- moved D18 3.28 mm to (134.8, 86.3)
- moved D19 3.28 mm to (134.8, 113.3)
- moved D20 3.28 mm to (134.8, 99.7)
- moved R30 3.28 mm to (134.9, 96.7)
- moved R31 3.28 mm to (134.9, 110.3)
- moved S1 3.28 mm to (144.6, 113.5)
- moved S2 3.28 mm to (144.6, 99.9)
- moved TH1 3.28 mm to (144.6, 86.5)
- moved U11 3.28 mm to (133.2, 79.7)
- moved JP1 3.24 mm to (137.9, 91.0), turned to 90 degrees
- moved R2 2.20 mm to (138.5, 136.4)
- moved D4 1.95 mm to (134.6, 136.4)
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- renumbered R24 to R21, R21 to R24, R27 to R26, R25 to R28, R26 to R29, R28 to R30, R29 to R31, R30 to R32, R31 to R33, R32 to R34, R33 to R35, R34 to R36, R35 to R37, R36 to R38, R37 to R39, R38 to R40, R39 to R41, R40 to R42, R41 to R43, R42 to R44, SHT1 to SHT40
Connections:
- JP1 pad 2: V3 -> Net-(JP1-B)
- Opto1 pad 1: +3.3V -> +5V
- R21 pad 1: +3.3V -> Net-(JP1-B)
- R21 pad 2: Net-(JP1-A) -> +3.3V
- TH1 pad 1: V3 -> Net-(JP1-A)
Routing:
- net +5V: track 145.0 -> 223.2 mm
- net +3.3V: track 318.0 -> 296.0 mm
- net Net-(JP1-A): track 1.95 -> 15.1 mm
- net SDA: track 115.1 -> 111.6 mm
- net SCL: track 117.7 -> 114.3 mm
- net V0: track 43.2 -> 46.5 mm
- net V3: track 19.6 -> 16.3 mm
- net Net-(JP1-B): track 0.00 -> 2.07 mm
- net 1Wire: track 118.2 -> 120.2 mm
- net Net-(D5-A): track 13.2 -> 14.9 mm
- net Net-(D15-A): track 6.20 -> 4.52 mm
- net CH7: track 101.3 -> 102.4 mm
- net In0: track 9.12 -> 8.19 mm
- net RX0: track 13.8 -> 14.5 mm
- net V1: track 43.8 -> 43.3 mm
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Other:
- board text added: "+5 IN GND"
- board text added: "Level 1 + -"
- board text added: "Level 2 + -"
- board text removed: "+Level1-"
- board text removed: "+Level2-"
- board text removed: "3V3"
