File: Habitat_V5/Habitat_V5.kicad_sch (KiCad schematic)
At the start: 102 parts, among them J1 Conn_01x03_Socket, J2 Conn_01x03_Socket, J3 Conn_01x12, J4 Conn_01x03_Socket, J5 Conn_01x04_Socket, K1 Relay_SPDT, Q1 PMOS, Q2 2N7002K, Q3 40N02, U1 XL1509-5V, U2 AP2112K-3.3, U3 PC817, U6 ESP32-WROOM-32

Commit message: Current update
Parts:
- C21: now not fitted; now left out of the parts list
- J2, J4, PWM1: footprint TerminalBlock:TerminalBlock_Xinya_XY308-2.54-3P_1x03_P2.54mm_Horizontal -> TerminalBlock_Phoenix:TerminalBlock_Phoenix_MKDS-1,5-3_1x03_P5.00mm_Horizontal
- J5: value Conn_01x04_Socket -> Conn_01x03_Socket; footprint TerminalBlock_Phoenix:TerminalBlock_Phoenix_MKDS-3-5-5.08_1x05_P5.08mm_Horizontal -> TerminalBlock_Phoenix:TerminalBlock_Phoenix_MKDS-1,5-3_1x03_P5.00mm_Horizontal; symbol Connector:Conn_01x05_Socket -> Connector:Conn_01x03_Socket
- Relay1: renamed from J1; footprint Connector_JST:JST_NV_B03P-NV_1x03_P5.00mm_Vertical -> TerminalBlock_Phoenix:TerminalBlock_Phoenix_MKDS-1,5-3_1x03_P5.00mm_Horizontal
- renumbered JP2 to JP1
Connections:
- net +5V: no longer C1.1, CD3.1, D1.1 (VDD)
- net +5V_H: now also C1.1, CD3.1, D1.1 (VDD)
- net GND: now also J5.3 (Pin_3); no longer J5.5 (Pin_5)
- net GPIO32: no longer J5.3 (Pin_3)
- net GPIO33: no longer J5.4 (Pin_4)
- net VCC: now also D4.2 (A), D5.1 (K), K1.A2
- net Vin: no longer D4.2 (A), D5.1 (K), K1.A1
- net at D5.2 (A), Q2.3 (D), R2.1: now also K1.A1; no longer K1.A2
- net at Relay1.1 (Pin_1): now also K1.14; no longer K1.12
- net at Relay1.3 (Pin_3): now also K1.12; no longer K1.14
Other:
- note added: "Display @ 0x3C"
- note removed: "Display I2C"
- moved on the sheet: C1, F1, K1, R7

Commit message: Updated PCB and Schematic
Parts:
- removed D14: SS14, Diode_SMD:D_SMA, symbol Diode:SS14
- removed J3: Conn_01x12, Connector_Phoenix_GMSTB:PhoenixContact_GMSTBVA_2,5_12-G-7,62_1x12_P7.62mm_Vertical, symbol Connector_Generic:Conn_01x12
- removed J5, PWM1: Conn_01x03_Socket, TerminalBlock_Phoenix:TerminalBlock_Phoenix_MKDS-1,5-3_1x03_P5.00mm_Horizontal, symbol Connector:Conn_01x03_Socket
- removed JP1: SolderJumper_3_Open, Jumper:SolderJumper-3_P2.0mm_Open_TrianglePad1.0x1.5mm, symbol Jumper:SolderJumper_3_Open
- removed Q3: 40N02, Package_TO_SOT_SMD:TO-252-2, symbol Transistor_FET:2N7002K
- removed R19: 2k2, Resistor_SMD:R_0805_2012Metric, symbol Device:R
- removed R20: 10k, Resistor_SMD:R_0805_2012Metric, symbol Device:R
- removed U6: ESP32-WROOM-32, RF_Module:ESP32-WROOM-32, symbol RF_Module:ESP32-WROOM-32
- added J1, J3, J4: Conn_01x04_Socket, Connector_Phoenix_MSTB:PhoenixContact_MSTBA_2,5_4-G-5,08_1x04_P5.08mm_Horizontal, symbol Connector:Conn_01x04_Socket
- added Opto1: Conn_01x02_Pin, Connector_Phoenix_MSTB:PhoenixContact_MSTBA_2,5_2-G-5,08_1x02_P5.08mm_Horizontal, symbol Connector:Conn_01x02_Pin
- added U6: ESP32-S3-WROOM-1, RF_Module:ESP32-S3-WROOM-1, symbol RF_Module:ESP32-S3-WROOM-1
- J2, Relay1: footprint TerminalBlock_Phoenix:TerminalBlock_Phoenix_MKDS-1,5-3_1x03_P5.00mm_Horizontal -> Connector_Phoenix_MSTB:PhoenixContact_MSTBA_2,5_3-G-5,08_1x03_P5.08mm_Horizontal
- J5: renamed from J4; footprint TerminalBlock_Phoenix:TerminalBlock_Phoenix_MKDS-1,5-3_1x03_P5.00mm_Horizontal -> Connector_Phoenix_MSTB:PhoenixContact_MSTBA_2,5_3-G-5,08_1x03_P5.08mm_Horizontal
- VDC1: footprint Connector_Phoenix_GMSTB:PhoenixContact_GMSTBVA_2,5_2-G-7,62_1x02_P7.62mm_Vertical -> Connector_Phoenix_MSTB:PhoenixContact_MSTBA_2,5_2-G-5,08_1x02_P5.08mm_Horizontal
- renumbered C21 to C18, C18 to C19, C19 to C20, C20 to C21, C25 to C22, C22 to C23, C23 to C24, C24 to C25, D15 to D14, R16 to R15, R15 to R16, R21 to R19, R9 to R7, R7 to R8, R8 to R9
Connections:
- net +3.3V: now also R13.2, Opto1.1 (Pin_1); no longer R13.1
- net 1Wire: now also U6.21 (IO13)
- net 3V3MCU: now also U6.2 (3V3)
- net GND: now also VDC1.1 (Pin_1), U6.1 (GND), U6.40 (GND), U6.41 (GND); no longer VDC1.2 (Pin_2)
- net In0: now also Opto1.2 (Pin_2)
- net NCH1: now also J1.2 (Pin_2)
- net NCH2: now also J1.4 (Pin_4)
- net NCH3: now also J3.2 (Pin_2)
- net NCH4: now also J3.4 (Pin_4)
- net NCH5: now also J4.2 (Pin_2)
- net NCH6: now also J4.4 (Pin_4)
- net Opto: now also U6.20 (IO12)
- net PCH1: now also J1.1 (Pin_1)
- net PCH2: now also J1.3 (Pin_3)
- net PCH3: now also J3.1 (Pin_1)
- net PCH4: now also J3.3 (Pin_3)
- net PCH5: now also J4.1 (Pin_1)
- net PCH6: now also J4.3 (Pin_3)
- net RX0: now also U6.36 (RXD0)
- net Relay: now also U6.23 (IO21)
- net SCL: now also U6.18 (IO10)
- net SDA: now also U6.19 (IO11)
- net TX0: now also U6.37 (TXD0)
- net Vin: now also VDC1.2 (Pin_2); no longer VDC1.1 (Pin_1)
- net EN: now reaches C7.1, R12.1, RST1.2
- net EN: now also U6.3 (EN)
- net PROG: now reaches C8.1, PROG1.2
- net PROG: now also R13.1, U6.27 (IO0); no longer R13.2
- net GPIO32 renamed GPIO11
- net GPIO11: now also U6.17 (IO9)
- net GPIO33 renamed GPIO10
- net GPIO10: now also U6.12 (IO8)
- new net CH1: U6.4 (IO4)
- new net CH2: U6.5 (IO5)
- new net CH3: U6.6 (IO6)
- new net CH4: U6.7 (IO7)
- new net CH5: U6.8 (IO15)
- new net CH6: U6.9 (IO16)
- new net CH7: U6.22 (IO14)
- new net EN_MASTER: U6.31 (IO38)
- no-connect marks 10 -> 11
Other:
- note added: "ESP32-S3-Wroom"
- note removed: "ESP32-Wroom"
- note removed: "Open Drain"
- moved on the sheet: C18, C22, C7, D11, D6, D7, J2, J5, R12, R13, R15, R8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

Commit message: Validation pre fab
Pls check
Parts:
- R11, R14, R16, R18, R19: LCSC C111857 -> C2683384
- R17: value 0R22 -> 0R25; LCSC C111857 -> C2932845
Connections:
- net +3.3V: now also J5.3 (Pin_3); no longer J5.1 (Pin_1)
- net GND: now also J5.1 (Pin_1); no longer J5.3 (Pin_3)
- net Neopixel: now also U6.15 (IO3)
Other:
- note added: "220mR 705mA"
- note added: "250mR 620mA"
- note added: "Vref=0.155V"
- moved on the sheet: J5
Changed lines of the file:
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@@
 	(wire
 		(pts
+			(xy 130.81 138.43) (xy 132.08 138.43)
+		)
+		(stroke
+			(width 0)
+			(type default)
+		)
+	)
+	(wire
+		(pts
 			(xy 78.74 232.41) (xy 92.71 232.41)
 		)
@@
 		)
 	)
+	(text "220mR\n705mA"
+		(exclude_from_sim no)
+		(at 96.012 110.49 0)
+		(effects
+			(font
+				(size 1.27 1.27)
+			)
+		)
+	)
+	(text "250mR\n620mA"
+		(exclude_from_sim no)
+		(at 97.028 241.808 0)
+		(effects
+			(font
+				(size 1.27 1.27)
+			)
+		)
+	)
+	(text "250mR\n620mA"
+		(exclude_from_sim no)
+		(at 96.52 189.484 0)
+		(effects
+			(font
+				(size 1.27 1.27)
+			)
+		)
+	)
+	(text "250mR\n620mA"
+		(exclude_from_sim no)
+		(at 96.52 215.138 0)
+		(effects
+			(font
+				(size 1.27 1.27)
+			)
+		)
+	)
 	(text "Status LED"
 		(exclude_from_sim no)
@@
 		)
 	)
+	(text "220mR\n705mA"
+		(exclude_from_sim no)
+		(at 96.52 137.922 0)
+		(effects
+			(font
+				(size 1.27 1.27)
+			)
+		)
+	)
 	(text "ESP32-S3-Wroom"
 		(exclude_from_sim no)
@@
 		)
 	)
+	(text "220mR\n705mA"
+		(exclude_from_sim no)
+		(at 96.266 162.814 0)
+		(effects
+			(font
+				(size 1.27 1.27)
+			)
+		)
+	)
 	(text "Voltage regulation"
 		(exclude_from_sim no)
@@
 		)
 	)
+	(text "Vref=0.155V"
+		(exclude_from_sim no)
+		(at 76.962 121.666 0)
+		(effects
+			(font
+				(size 1.27 1.27)
+			)
+		)
+	)
 	(text "Opto"
 		(exclude_from_sim no)
@@
 	(global_label "Neopixel"
 		(shape input)
-		(at 129.54 133.35 180)
+		(at 130.81 138.43 180)
 		(fields_autoplaced yes)
 		(effects
@@
 		)
 		(property "Intersheetrefs" "${INTERSHEET_REFS}"
-			(at 118.451 133.35 0)
+			(at 119.721 138.43 0)
 			(effects
 				(font
@@
 			)
 		)
-		(property "LCSC" "C111857"
+		(property "LCSC" "C2683384"
 			(at 90.17 241.3 90)
 			(effects
@@
 			)
 		)
-		(property "Value" "0R22"
+		(property "Value" "0R25"
 			(at 87.884 189.23 90)
 			(effects
@@
 			)
 		)
-		(property "LCSC" "C111857"
+		(property "LCSC" "C2932845"
 			(at 90.17 189.23 90)
 			(effects
@@
 			)
 		)
-		(property "LCSC" "C111857"
+		(property "LCSC" "C2683384"
 			(at 90.17 110.49 90)
 			(effects
@@
 			)
 		)
-		(property "LCSC" "C111857"
+		(property "LCSC" "C2683384"
 			(at 90.17 214.63 90)
 			(effects
@@
 	(symbol
 		(lib_id "Connector:Conn_01x03_Socket")
-		(at 170.18 231.14 0)
-		(mirror y)
+		(at 170.18 231.14 180)
 		(unit 1)
 		(exclude_from_sim no)
@@
 		(dnp no)
 		(property "Reference" "J5"
-			(at 173.228 224.282 0)
+			(at 170.688 224.79 0)
 			(effects
 				(font
@@
 		)
 		(property "Value" "Conn_01x03_Socket"
-			(at 168.91 232.4099 0)
+			(at 168.91 229.8701 0)
 			(effects
 				(font
@@
 			)
 		)
-		(property "LCSC" "C111857"
+		(property "LCSC" "C2683384"
 			(at 90.17 137.16 90)
 			(effects
@@
 			)
 		)
-		(property "LCSC" "C111857"
+		(property "LCSC" "C2683384"
 			(at 90.17 162.56 90)
 			(effects

Commit message: Review for production
Parts:
- R18: value 0R22 -> 0R25; LCSC C2683384 -> C2932845
- renumbered VDC2 to VDC1, VDC1 to VDC2
Connections:
- net Neopixel: now also U6.10 (IO17); no longer U6.15 (IO3)
- net GPIO10 renamed GPIO8
- net GPIO11 renamed GPIO9
Changed lines of the file:
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@@
 	(wire
 		(pts
-			(xy 130.81 138.43) (xy 132.08 138.43)
-		)
-		(stroke
-			(width 0)
-			(type default)
-		)
-	)
-	(wire
-		(pts
 			(xy 78.74 232.41) (xy 92.71 232.41)
 		)
@@
 		)
 	)
+	(text "250mR\n620mA"
+		(exclude_from_sim no)
+		(at 96.266 163.068 0)
+		(effects
+			(font
+				(size 1.27 1.27)
+			)
+		)
+	)
 	(text "WLED"
 		(exclude_from_sim no)
@@
 		)
 	)
-	(text "220mR\n705mA"
-		(exclude_from_sim no)
-		(at 96.266 162.814 0)
-		(effects
-			(font
-				(size 1.27 1.27)
-			)
-		)
-	)
 	(text "Voltage regulation"
 		(exclude_from_sim no)
@@
 		)
 	)
-	(global_label "GPIO11"
+	(global_label "GPIO9"
 		(shape input)
 		(at 129.54 153.67 180)
@@
 		)
 		(property "Intersheetrefs" "${INTERSHEET_REFS}"
-			(at 119.6605 153.67 0)
+			(at 120.87 153.67 0)
 			(effects
 				(font
@@
 		)
 	)
-	(global_label "GPIO11"
+	(global_label "GPIO9"
 		(shape input)
 		(at 68.58 78.74 180)
@@
 		)
 		(property "Intersheetrefs" "${INTERSHEET_REFS}"
-			(at 58.7005 78.74 0)
+			(at 59.91 78.74 0)
 			(effects
 				(font
@@
 		)
 	)
-	(global_label "GPIO10"
+	(global_label "GPIO8"
 		(shape input)
 		(at 129.54 151.13 180)
@@
 		)
 		(property "Intersheetrefs" "${INTERSHEET_REFS}"
-			(at 119.6605 151.13 0)
+			(at 120.87 151.13 0)
 			(effects
 				(font
@@
 	(global_label "Neopixel"
 		(shape input)
-		(at 130.81 138.43 180)
+		(at 162.56 130.81 0)
 		(fields_autoplaced yes)
 		(effects
@@
 				(size 1.27 1.27)
 			)
-			(justify right)
+			(justify left)
 		)
 		(property "Intersheetrefs" "${INTERSHEET_REFS}"
-			(at 119.721 138.43 0)
+			(at 173.649 130.81 0)
 			(effects
 				(font
 					(size 1.27 1.27)
 				)
-				(justify right)
+				(justify left)
 				(hide yes)
 			)
@@
 		)
 	)
-	(global_label "GPIO10"
+	(global_label "GPIO8"
 		(shape input)
 		(at 68.58 81.28 180)
@@
 		)
 		(property "Intersheetrefs" "${INTERSHEET_REFS}"
-			(at 58.7005 81.28 0)
+			(at 59.91 81.28 0)
 			(effects
 				(font
@@
 		(dnp no)
 		(fields_autoplaced yes)
-		(property "Reference" "VDC2"
+		(property "Reference" "VDC1"
 			(at 105.41 67.31 0)
 			(effects
@@
 			(project "Habitat_V5"
 				(path "/5da8ef61-9b4a-4ae5-94b1-3a318860cb02"
-					(reference "VDC2")
+					(reference "VDC1")
 					(unit 1)
 				)
@@
 	)
 	(symbol
-		(lib_id "Device:R")
-		(at 90.17 214.63 0)
-		(unit 1)
-		(exclude_from_sim no)
-		(in_bom yes)
-		(on_board yes)
-		(dnp no)
-		(property "Reference" "R18"
-			(at 90.17 214.63 90)
-			(effects
-				(font
-					(size 1.27 1.27)
-				)
-			)
-		)
-		(property "Value" "0R22"
-			(at 87.884 214.63 90)
-			(effects
-				(font
-					(size 1.27 1.27)
-				)
-			)
-		)
-		(property "Footprint" "Resistor_SMD:R_1206_3216Metric"
-			(at 88.392 214.63 90)
-			(effects
-				(font
-					(size 1.27 1.27)
-				)
-				(hide yes)
-			)
-		)
-		(property "Datasheet" "~"
-			(at 90.17 214.63 0)
-			(effects
-				(font
-					(size 1.27 1.27)
-				)
-				(hide yes)
-			)
-		)
-		(property "Description" "Resistor"
-			(at 90.17 214.63 0)
-			(effects
-				(font
-					(size 1.27 1.27)
-				)
-				(hide yes)
-			)
-		)
-		(property "LCSC" "C2683384"
-			(at 90.17 214.63 90)
-			(effects
-				(font
-					(size 1.27 1.27)
-				)
-				(hide yes)
-			)
-		)
-		(property "ASSEMBLY" ""
-			(at 90.17 214.63 0)
-			(effects
-				(font
-					(size 1.27 1.27)
-				)
-				(hide yes)
-			)
-		)
-		(property "PART NUMBER" ""
-			(at 90.17 214.63 0)
-			(effects
-				(font
-					(size 1.27 1.27)
-				)
-				(hide yes)
-			)
-		)
-		(property "SUPPLIER 1" ""
-			(at 90.17 214.63 0)
-			(effects
-				(font
-					(size 1.27 1.27)
-				)
-				(hide yes)
-			)
-		)
-		(property "SUPPLIER 2" ""
-			(at 90.17 214.63 0)
-			(effects
-				(font
-					(size 1.27 1.27)
-				)
-				(hide yes)
-			)
-		)
-		(property "SUPPLIER 3" ""
-			(at 90.17 214.63 0)
-			(effects
-				(font
-					(size 1.27 1.27)
-				)
-				(hide yes)
-			)
-		)
-		(property "SUPPLIER PART NUMBER 1" ""
-			(at 90.17 214.63 0)
-			(effects
-				(font
-					(size 1.27 1.27)
-				)
-				(hide yes)
-			)
-		)
-		(property "SUPPLIER PART NUMBER 2" ""
-			(at 90.17 214.63 0)
-			(effects
-				(font
-					(size 1.27 1.27)
-				)
-				(hide yes)
-			)
-		)
-		(property "SUPPLIER PART NUMBER 3" ""
-			(at 90.17 214.63 0)
-			(effects
-				(font
-					(size 1.27 1.27)
-				)
-				(hide yes)
-			)
-		)
-		(property "TYPE" ""
-			(at 90.17 214.63 0)
-			(effects
-				(font
-					(size 1.27 1.27)
-				)
-				(hide yes)
-			)
-		)
-		(pin "1"
-		)
-		(pin "2"
-		)
-		(instances
-			(project "Habitat_V5"
-				(path "/5da8ef61-9b4a-4ae5-94b1-3a318860cb02"
-					(reference "R18")
-					(unit 1)
-				)
-			)
-		)
-	)
-	(symbol
 		(lib_id "power:GND")
 		(at 62.23 49.53 0)
@@
 	)
 	(symbol
+		(lib_id "Device:R")
+		(at 90.17 214.63 0)
+		(unit 1)
+		(exclude_from_sim no)
+		(in_bom yes)
+		(on_board yes)
+		(dnp no)
+		(property "Reference" "R18"
+			(at 90.17 214.63 90)
+			(effects
+				(font
+					(size 1.27 1.27)
+				)
+			)
+		)
+		(property "Value" "0R25"
+			(at 87.884 214.63 90)
+			(effects
+				(font
+					(size 1.27 1.27)
+				)
+			)
+		)
+		(property "Footprint" "Resistor_SMD:R_1206_3216Metric"
+			(at 88.392 214.63 90)
+			(effects
+				(font
+					(size 1.27 1.27)
+				)
+				(hide yes)
+			)
+		)
+		(property "Datasheet" "~"
+			(at 90.17 214.63 0)
+			(effects
+				(font
+					(size 1.27 1.27)
+				)
+				(hide yes)
+			)
+		)
+		(property "Description" "Resistor"
+			(at 90.17 214.63 0)
+			(effects
+				(font
+					(size 1.27 1.27)
+				)
+				(hide yes)
+			)
+		)
+		(property "LCSC" "C2932845"
+			(at 90.17 214.63 90)
+			(effects
+				(font
+					(size 1.27 1.27)
+				)
+				(hide yes)
+			)
+		)
+		(property "ASSEMBLY" ""
+			(at 90.17 214.63 0)
+			(effects
+				(font
+					(size 1.27 1.27)
+				)
+				(hide yes)
+			)
+		)
+		(property "PART NUMBER" ""
+			(at 90.17 214.63 0)
+			(effects
+				(font
+					(size 1.27 1.27)
+				)
+				(hide yes)
+			)
+		)
+		(property "SUPPLIER 1" ""
+			(at 90.17 214.63 0)
+			(effects
+				(font
+					(size 1.27 1.27)
+				)
+				(hide yes)
+			)
+		)
+		(property "SUPPLIER 2" ""
+			(at 90.17 214.63 0)
+			(effects
+				(font
+					(size 1.27 1.27)
+				)
+				(hide yes)
+			)
+		)
+		(property "SUPPLIER 3" ""
+			(at 90.17 214.63 0)
+			(effects
+				(font
+					(size 1.27 1.27)
+				)
+				(hide yes)
+			)
+		)
+		(property "SUPPLIER PART NUMBER 1" ""
+			(at 90.17 214.63 0)
+			(effects
+				(font
+					(size 1.27 1.27)
+				)
+				(hide yes)
+			)
+		)
+		(property "SUPPLIER PART NUMBER 2" ""
+			(at 90.17 214.63 0)
+			(effects
+				(font
+					(size 1.27 1.27)
+				)
+				(hide yes)
+			)
+		)
+		(property "SUPPLIER PART NUMBER 3" ""
+			(at 90.17 214.63 0)
+			(effects
+				(font
+					(size 1.27 1.27)
+				)
+				(hide yes)
+			)
+		)
+		(property "TYPE" ""
+			(at 90.17 214.63 0)
+			(effects
+				(font
+					(size 1.27 1.27)
+				)
+				(hide yes)
+			)
+		)
+		(pin "1"
+		)
+		(pin "2"
+		)
+		(instances
+			(project "Habitat_V5"
+				(path "/5da8ef61-9b4a-4ae5-94b1-3a318860cb02"
+					(reference "R18")
+					(unit 1)
+				)
+			)
+		)
+	)
+	(symbol
 		(lib_id "Connector:Conn_01x03_Socket")
 		(at 170.18 231.14 180)
@@
 		(on_board yes)
 		(dnp no)
-		(property "Reference" "VDC1"
+		(property "Reference" "VDC2"
 			(at 90.678 80.518 0)
 			(effects
@@
 			(project "Habitat_V5"
 				(path "/5da8ef61-9b4a-4ae5-94b1-3a318860cb02"
-					(reference "VDC1")
+					(reference "VDC2")
 					(unit 1)
 				)

Commit message: Files for production
Parts:
- Opto1: value Conn_01x02_Pin -> Conn_01x03_Pin; footprint Connector_Phoenix_MSTB:PhoenixContact_MSTBA_2,5_2-G-5,08_1x02_P5.08mm_Horizontal -> Connector_Phoenix_MSTB:PhoenixContact_MSTBA_2,5_3-G-5,08_1x03_P5.08mm_Horizontal; symbol Connector:Conn_01x02_Pin -> Connector:Conn_01x03_Pin
Connections:
- net +3.3V: no longer Opto1.1 (Pin_1)
- net +5V: now also Opto1.1 (Pin_1)
- net GND: now also Opto1.3 (Pin_3)
Changed lines of the file:
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@@
 	(wire
 		(pts
-			(xy 130.81 68.58) (xy 128.27 68.58)
+			(xy 129.54 64.77) (xy 127 64.77)
 		)
 		(stroke
@@
 	(global_label "In0"
 		(shape input)
-		(at 128.27 71.12 0)
+		(at 127 67.31 0)
 		(fields_autoplaced yes)
 		(effects
@@
 		)
 		(property "Intersheetrefs" "${INTERSHEET_REFS}"
-			(at 134.2185 71.12 0)
+			(at 132.9485 67.31 0)
 			(effects
 				(font
@@
 	)
 	(symbol
-		(lib_id "power:+3.3V")
-		(at 130.81 68.58 0)
-		(unit 1)
-		(exclude_from_sim no)
-		(in_bom yes)
-		(on_board yes)
-		(dnp no)
-		(property "Reference" "#PWR24"
-			(at 130.81 72.39 0)
-			(effects
-				(font
-					(size 1.27 1.27)
-				)
-				(hide yes)
-			)
-		)
-		(property "Value" "+3.3V"
-			(at 135.382 67.31 0)
-			(effects
-				(font
-					(size 1.27 1.27)
-				)
-			)
-		)
-		(property "Footprint" ""
-			(at 130.81 68.58 0)
-			(effects
-				(font
-					(size 1.27 1.27)
-				)
-				(hide yes)
-			)
-		)
-		(property "Datasheet" ""
-			(at 130.81 68.58 0)
-			(effects
-				(font
-					(size 1.27 1.27)
-				)
-				(hide yes)
-			)
-		)
-		(property "Description" "Power symbol creates a global label with name \"+3.3V\""
-			(at 130.81 68.58 0)
-			(effects
-				(font
-					(size 1.27 1.27)
-				)
-				(hide yes)
-			)
-		)
-		(pin "1"
-		)
-		(instances
-			(project "Habitat_V5"
-				(path "/5da8ef61-9b4a-4ae5-94b1-3a318860cb02"
-					(reference "#PWR24")
-					(unit 1)
-				)
-			)
-		)
-	)
-	(symbol
 		(lib_id "Device:C_Polarized")
 		(at 78.74 187.96 0)
@@
 	)
 	(symbol
-		(lib_id "Connector:Conn_01x02_Pin")
-		(at 123.19 68.58 0)
+		(lib_id "Connector:Conn_01x03_Pin")
+		(at 121.92 67.31 0)
 		(unit 1)
 		(exclude_from_sim no)
@@
 		(dnp no)
 		(property "Reference" "Opto1"
-			(at 123.698 65.532 0)
+			(at 123.698 59.69 0)
 			(effects
 				(font
@@
 			)
 		)
-		(property "Value" "Conn_01x02_Pin"
-			(at 123.825 66.04 0)
+		(property "Value" "Conn_01x03_Pin"
+			(at 122.555 64.77 0)
 			(effects
 				(font
@@
 			)
 		)
-		(property "Footprint" "Connector_Phoenix_MSTB:PhoenixContact_MSTBA_2,5_2-G-5,08_1x02_P5.08mm_Horizontal"
-			(at 123.19 68.58 0)
+		(property "Footprint" "Connector_Phoenix_MSTB:PhoenixContact_MSTBA_2,5_3-G-5,08_1x03_P5.08mm_Horizontal"
+			(at 121.92 67.31 0)
 			(effects
 				(font
@@
 		)
 		(property "Datasheet" "~"
-			(at 123.19 68.58 0)
+			(at 121.92 67.31 0)
 			(effects
 				(font
@@
 			)
 		)
-		(property "Description" "Generic connector, single row, 01x02, script generated"
-			(at 123.19 68.58 0)
+		(property "Description" "Generic connector, single row, 01x03, script generated"
+			(at 121.92 67.31 0)
 			(effects
 				(font
@@
 		)
 		(property "LCSC" "1"
-			(at 123.19 68.58 0)
+			(at 121.92 67.31 0)
 			(effects
 				(font
@@
 		)
 		(property "ASSEMBLY" ""
-			(at 123.19 68.58 0)
+			(at 121.92 67.31 0)
 			(effects
 				(font
@@
 		)
 		(property "PART NUMBER" ""
-			(at 123.19 68.58 0)
+			(at 121.92 67.31 0)
 			(effects
 				(font
@@
 		)
 		(property "SUPPLIER 1" ""
-			(at 123.19 68.58 0)
+			(at 121.92 67.31 0)
 			(effects
 				(font
@@
 		)
 		(property "SUPPLIER 2" ""
-			(at 123.19 68.58 0)
+			(at 121.92 67.31 0)
 			(effects
 				(font
@@
 		)
 		(property "SUPPLIER 3" ""
-			(at 123.19 68.58 0)
+			(at 121.92 67.31 0)
 			(effects
 				(font
@@
 		)
 		(property "SUPPLIER PART NUMBER 1" ""
-			(at 123.19 68.58 0)
+			(at 121.92 67.31 0)
 			(effects
 				(font
@@
 		)
 		(property "SUPPLIER PART NUMBER 2" ""
-			(at 123.19 68.58 0)
+			(at 121.92 67.31 0)
 			(effects
 				(font
@@
 		)
 		(property "SUPPLIER PART NUMBER 3" ""
-			(at 123.19 68.58 0)
+			(at 121.92 67.31 0)
 			(effects
 				(font
@@
 		)
 		(property "TYPE" ""
-			(at 123.19 68.58 0)
+			(at 121.92 67.31 0)
 			(effects
 				(font
@@
 		(pin "1"
 		)
+		(pin "3"
+		)
 		(instances
 			(project "Habitat_V5"
@@
 	)
 	(symbol
+		(lib_id "power:GND")
+		(at 127 69.85 0)
+		(unit 1)
+		(exclude_from_sim no)
+		(in_bom yes)
+		(on_board yes)
+		(dnp no)
+		(fields_autoplaced yes)
+		(property "Reference" "#PWR145"
+			(at 127 76.2 0)
+			(effects
+				(font
+					(size 1.27 1.27)
+				)
+				(hide yes)
+			)
+		)
+		(property "Value" "GND"
+			(at 127 74.93 0)
+			(effects
+				(font
+					(size 1.27 1.27)
+				)
+			)
+		)
+		(property "Footprint" ""
+			(at 127 69.85 0)
+			(effects
+				(font
+					(size 1.27 1.27)
+				)
+				(hide yes)
+			)
+		)
+		(property "Datasheet" ""
+			(at 127 69.85 0)
+			(effects
+				(font
+					(size 1.27 1.27)
+				)
+				(hide yes)
+			)
+		)
+		(property "Description" "Power symbol creates a global label with name \"GND\" , ground"
+			(at 127 69.85 0)
+			(effects
+				(font
+					(size 1.27 1.27)
+				)
+				(hide yes)
+			)
+		)
+		(pin "1"
+		)
+		(instances
+			(project "Habitat_V5"
+				(path "/5da8ef61-9b4a-4ae5-94b1-3a318860cb02"
+					(reference "#PWR145")
+					(unit 1)
+				)
+			)
+		)
+	)
+	(symbol
 		(lib_id "Device:D_Zener")
 		(at 31.75 38.1 180)
@@
 					(unit 1)
 				)
+			)
+		)
+	)
+	(symbol
+		(lib_id "power:+5V")
+		(at 129.54 64.77 0)
+		(unit 1)
+		(exclude_from_sim no)
+		(in_bom yes)
+		(on_board yes)
+		(dnp no)
+		(property "Reference" "#PWR24"
+			(at 129.54 68.58 0)
+			(effects
+				(font
+					(size 1.27 1.27)
+				)
+				(hide yes)
+			)
+		)
+		(property "Value" "+5V"
+			(at 129.54 60.452 0)
+			(effects
+				(font
+					(size 1.27 1.27)
+				)
+			)
+		)
+		(property "Footprint" ""
+			(at 129.54 64.77 0)
+			(effects
+				(font
+					(size 1.27 1.27)
+				)
+				(hide yes)
+			)
+		)
+		(property "Datasheet" ""
+			(at 129.54 64.77 0)
+			(effects
+				(font
+					(size 1.27 1.27)
+				)
+				(hide yes)
+			)
+		)
+		(property "Description" "Power symbol creates a global label with name \"+5V\""
+			(at 129.54 64.77 0)
+			(effects
+				(font
+					(size 1.27 1.27)
+				)
+				(hide yes)
+			)
+		)
+		(pin "1"
+		)
+		(instances
+			(project "Habitat_V5"
+				(path "/5da8ef61-9b4a-4ae5-94b1-3a318860cb02"
+					(reference "#PWR24")
+					(unit 1)
+				)
